File: clkdiv.kicad_sch (KiCad schematic)
At the start: 57 parts, among them J1 CLK IN, J10 CLK OUT 7, J11 CLK OUT 8, J2 RST, J3 EURORACK POWER, J4 CLK OUT 1, J5 CLK OUT 2, J6 CLK OUT 3, J7 CLK OUT 4, J8 CLK OUT 5, J9 CLK OUT 6, Q1 2N3904, Q2 2N3904, SW1 SW_Push, U1 L78L05_TO92, U2 PROMICRO

Commit message: Move GND symbol and remove unused diode definition
Parts:
- removed D1, D2: 1N4148, Diode_THT:D_DO-35_SOD27_P7.62mm_Horizontal, symbol Diode:1N4148
Connections:
- net GND: now also Q1.1 (E), Q2.1 (E)
Changed lines of the file:
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@@
 	(symbol
 		(lib_id "power:GND")
-		(at 83.82 48.26 0)
+		(at 83.82 40.64 0)
 		(mirror y)
 		(unit 1)
@@
 		(fields_autoplaced yes)
 		(property "Reference" "#PWR017"
-			(at 83.82 54.61 0)
+			(at 83.82 46.99 0)
 			(effects
 				(font
@@
 		)
 		(property "Value" "GND"
-			(at 83.82 53.34 0)
+			(at 83.82 45.72 0)
 			(effects
 				(font
@@
 		)
 		(property "Footprint" ""
-			(at 83.82 48.26 0)
+			(at 83.82 40.64 0)
 			(effects
 				(font
@@
 		)
 		(property "Datasheet" ""
-			(at 83.82 48.26 0)
+			(at 83.82 40.64 0)
 			(effects
 				(font
@@
 		)
 		(property "Description" "Power symbol creates a global label with name \"GND\" , ground"
-			(at 83.82 48.26 0)
+			(at 83.82 40.64 0)
 			(effects
 				(font
@@
 	)
 	(symbol
-		(lib_id "Diode:1N4148")
-		(at 83.82 86.36 270)
-		(unit 1)
-		(exclude_from_sim no)
-		(in_bom yes)
-		(on_board yes)
-		(dnp no)
-		(fields_autoplaced yes)
-		(property "Reference" "D2"
-			(at 86.36 85.0899 90)
-			(effects
-				(font
-					(size 1.27 1.27)
-				)
-				(justify left)
-			)
-		)
-		(property "Value" "1N4148"
-			(at 86.36 87.6299 90)
-			(effects
-				(font
-					(size 1.27 1.27)
-				)
-				(justify left)
-			)
-		)
-		(property "Footprint" "Diode_THT:D_DO-35_SOD27_P7.62mm_Horizontal"
-			(at 83.82 86.36 0)
-			(effects
-				(font
-					(size 1.27 1.27)
-				)
-				(hide yes)
-			)
-		)
-		(property "Datasheet" "https://assets.nexperia.com/documents/data-sheet/1N4148_1N4448.pdf"
-			(at 83.82 86.36 0)
-			(effects
-				(font
-					(size 1.27 1.27)
-				)
-				(hide yes)
-			)
-		)
-		(property "Description" "100V 0.15A standard switching diode, DO-35"
-			(at 83.82 86.36 0)
-			(effects
-				(font
-					(size 1.27 1.27)
-				)
-				(hide yes)
-			)
-		)
-		(property "Sim.Device" "D"
-			(at 83.82 86.36 0)
-			(effects
-				(font
-					(size 1.27 1.27)
-				)
-				(hide yes)
-			)
-		)
-		(property "Sim.Pins" "1=K 2=A"
-			(at 83.82 86.36 0)
-			(effects
-				(font
-					(size 1.27 1.27)
-				)
-				(hide yes)
-			)
-		)
-		(pin "1"
-		)
-		(pin "2"
-		)
-		(instances
-			(project "clkdiv"
-				(path "/11ddf9e5-4dd0-439a-af1c-50fd056d6733"
-					(reference "D2")
-					(unit 1)
-				)
-			)
-		)
-	)
-	(symbol
 		(lib_id "Regulator_Linear:L78L05_TO92")
 		(at 123.19 115.57 0)
@@
 	(symbol
 		(lib_id "power:GND")
-		(at 83.82 90.17 0)
+		(at 83.82 82.55 0)
 		(mirror y)
 		(unit 1)
@@
 		(fields_autoplaced yes)
 		(property "Reference" "#PWR019"
-			(at 83.82 96.52 0)
+			(at 83.82 88.9 0)
 			(effects
 				(font
@@
 		)
 		(property "Value" "GND"
-			(at 83.82 95.25 0)
+			(at 83.82 87.63 0)
 			(effects
 				(font
@@
 		)
 		(property "Footprint" ""
-			(at 83.82 90.17 0)
+			(at 83.82 82.55 0)
 			(effects
 				(font
@@
 		)
 		(property "Datasheet" ""
-			(at 83.82 90.17 0)
+			(at 83.82 82.55 0)
 			(effects
 				(font
@@
 		)
 		(property "Description" "Power symbol creates a global label with name \"GND\" , ground"
-			(at 83.82 90.17 0)
+			(at 83.82 82.55 0)
 			(effects
 				(font
@@
 					(unit 1)
 				)
-			)
-		)
-	)
-	(symbol
-		(lib_id "Diode:1N4148")
-		(at 83.82 44.45 270)
-		(unit 1)
-		(exclude_from_sim no)
-		(in_bom yes)
-		(on_board yes)
-		(dnp no)
-		(fields_autoplaced yes)
-		(property "Reference" "D1"
-			(at 86.36 43.1799 90)
-			(effects
-				(font
-					(size 1.27 1.27)
-				)
-				(justify left)
-			)
-		)
-		(property "Value" "1N4148"
-			(at 86.36 45.7199 90)
-			(effects
-				(font
-					(size 1.27 1.27)
-				)
-				(justify left)
-			)
-		)
-		(property "Footprint" "Diode_THT:D_DO-35_SOD27_P7.62mm_Horizontal"
-			(at 83.82 44.45 0)
-			(effects
-				(font
-					(size 1.27 1.27)
-				)
-				(hide yes)
-			)
-		)
-		(property "Datasheet" "https://assets.nexperia.com/documents/data-sheet/1N4148_1N4448.pdf"
-			(at 83.82 44.45 0)
-			(effects
-				(font
-					(size 1.27 1.27)
-				)
-				(hide yes)
-			)
-		)
-		(property "Description" "100V 0.15A standard switching diode, DO-35"
-			(at 83.82 44.45 0)
-			(effects
-				(font
-					(size 1.27 1.27)
-				)
-				(hide yes)
-			)
-		)
-		(property "Sim.Device" "D"
-			(at 83.82 44.45 0)
-			(effects
-				(font
-					(size 1.27 1.27)
-				)
-				(hide yes)
-			)
-		)
-		(property "Sim.Pins" "1=K 2=A"
-			(at 83.82 44.45 0)
-			(effects
-				(font
-					(size 1.27 1.27)
-				)
-				(hide yes)
-			)
-		)
-		(pin "1"
-		)
-		(pin "2"
-		)
-		(instances
-			(project ""
-				(path "/11ddf9e5-4dd0-439a-af1c-50fd056d6733"
-					(reference "D1")
-					(unit 1)
-				)
